File: Pancake pcb/Pancake.kicad_pcb (KiCad board)
At the start: 2 copper layers, 246 x 83 mm, 87 parts, among them J1 Conn_01x04, U1 Frood

Commit message: Many change
Parts:
- added REF**: Stabilizer_Cherry_MX_2.00u, PCM_Mounting_Keyboard_Stabilizer:Stabilizer_Cherry_MX_2.00u, F.Cu at (115.7, 90.2)
- added REF**: Stabilizer_Cherry_MX_2.00u, PCM_Mounting_Keyboard_Stabilizer:Stabilizer_Cherry_MX_2.00u, F.Cu at (172.9, 90.2)
- moved D38 8.10 mm to (132.6, 92.6)
- moved D40 8.10 mm to (189.7, 92.6)
- moved D33 2.38 mm to (214.9, 74.0)
- moved MX32 2.38 mm to (187.2, 72.0)
- moved MX35 2.38 mm to (246.7, 72.0)
- moved D26 2.38 mm to (81.6, 74.0)
- moved D27 2.38 mm to (100.6, 74.0)
- moved MX26 2.38 mm to (72.9, 72.0)
- moved D25 2.38 mm to (57.8, 74.0)
- moved MX25 2.38 mm to (49.1, 72.0)
- moved D28 2.38 mm to (119.7, 74.0)
- moved D29 2.38 mm to (138.7, 74.0)
- moved D30 2.38 mm to (157.8, 74.0)
- moved D31 2.38 mm to (176.8, 74.0)
- moved D32 2.38 mm to (195.9, 74.0)
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Routing:
- net Net-(D38-A): track 8.27 -> 16.4 mm
- net Net-(D40-A): track 8.27 -> 16.4 mm
- net Col6: track 151.3 -> 143.4 mm
- net Col0: track 251.4 -> 254.2 mm
- net Col9: track 92.7 -> 95.4 mm
- net Col2: track 225.8 -> 223.4 mm
- net Col1: track 248.1 -> 250.4 mm
- net Col5: track 169.9 -> 168.0 mm
- net Col8: track 121.5 -> 119.5 mm
- net Col4: track 202.2 -> 200.5 mm
- net Col7: track 158.2 -> 157.0 mm
- net Row2: track 206.8 -> 205.9 mm
- net Col11: track 54.7 -> 55.3 mm

Commit message: Modification complète du PCB et fichier de production
Flemme de faire en anglais au pire google traduction ça existe 😭

J'ai complètement refait le pcb pour mettre les diodes derrière et donc refait tout le routing, en plus de ça j'ai fait les fichier pour faire produire le pcb par jlcpcb donc vous pourrez aussi le produire.
Parts:
- D1, D10, D11, D12, D13, D14, D15, D16, D17, D18, D19, D2, D20, D21, D22, D23, D24, D25, D26, D27, D28, D29, D3, D30, D31, D32, D33, D34, D35, D36, D37, D38, D39, D4, D40, D41, D42, D5, D6, D7, D8, D9: moved to B.Cu
- moved D42 17.2 mm to (231.4, 92.6)
- moved D38 8.26 mm to (124.3, 92.7)
- moved D40 8.26 mm to (181.5, 92.6)
Routing:
- net Col6: track 143.4 -> 125.9 mm, vias 0 -> 2
- net Col7: track 157.0 -> 143.7 mm, vias 0 -> 2
- net Net-(D40-A): track 16.4 -> 8.11 mm
- net Net-(D38-A): track 16.4 -> 8.14 mm
- net GND: track 8.13 -> 0.00 mm
- net Net-(D42-A): track 15.7 -> 8.02 mm
- net Row3: track 176.9 -> 183.4 mm
- net Col8: track 119.5 -> 114.5 mm, vias 0 -> 2
- net Col9: track 95.4 -> 92.1 mm
- net Col2: track 223.4 -> 226.0 mm
- net RAW: track 15.0 -> 17.5 mm, vias 0 -> 1
- net Col5: track 168.0 -> 170.0 mm
- net Col4: track 200.5 -> 202.0 mm
- net Row0: track 261.8 -> 260.9 mm
- net Col1: track 250.4 -> 251.1 mm
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