File: Pancake pcb/Pancake.kicad_pcb (KiCad board)
At the start: 2 copper layers, 246 x 83 mm, 89 parts, among them J1 Conn_01x04, U1 Frood

Commit message: PCB last modification
Parts:
- added G***: LOGO, LOGO, F.Cu at (41.3, 100.4)
- moved G*** 11.3 mm to (35.0, 87.3)
