File: PancakeXXL PCB/PancakeXXL V2-rounded.kicad_pcb (KiCad board)
At the start: 2 copper layers, 246 x 83 mm, 119 parts, among them J1 Conn_01x04, SW1 Reset, SW2 Boot, U1 XC6206PxxxMR, U2 RP2040, U3 W25Q128JVS, Y1 ABM8-272-T3

Commit message: C'était pas droit avant, mainteant le pcb et le KLE l'ai faut que je fasse la plate et la case mtn
Parts:
- U1: footprint Package_TO_SOT_SMD:SOT-223-3_TabPin2 -> Package_TO_SOT_SMD:SOT-23-3
- moved C1 60.7 mm to (258.0, 77.2), turned to 0 degrees
- moved D36 2.27 mm to (76.7, 92.6)
- moved D38 2.27 mm to (126.6, 92.7)
- moved D39 2.27 mm to (155.3, 92.6)
- moved D40 2.27 mm to (183.7, 92.6)
- moved D41 2.27 mm to (212.5, 92.6)
- moved D42 2.27 mm to (233.6, 92.6)
- moved MX36 2.27 mm to (68.0, 91.0)
- moved MX39 2.27 mm to (146.6, 91.0)
- moved MX40 2.27 mm to (175.1, 91.0)
- moved MX42 2.27 mm to (225.2, 91.0)
- moved REF** 2.27 mm to (175.1, 90.2)
- moved D37 2.27 mm to (98.2, 92.6)
- moved MX37 2.27 mm to (89.4, 91.0)
- moved MX38 2.27 mm to (118.0, 91.0)
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Routing:
- net Col5: track 181.6 -> 177.2 mm
- net VBUS: track 81.3 -> 85.2 mm
- net Col9: track 113.2 -> 109.9 mm
- net Col4: track 218.0 -> 214.7 mm
- net Col8: track 123.4 -> 120.2 mm
- net Col7: track 155.9 -> 153.0 mm
- net Col2: track 242.0 -> 240.0 mm
- net +3V3: track 68.5 -> 66.7 mm
- net Col1: track 264.0 -> 262.9 mm
- net Row3: track 176.6 -> 175.6 mm
- net Col3: track 214.0 -> 214.8 mm

Commit message: Rectification KLE, 3D
J'ai refait tout le design pour que cette fois-ci tout soit bien droit
Parts:
- moved C1 5.91 mm to (261.0, 72.1), turned to 180 degrees
- moved G*** 0.18 mm to (35.2, 87.3)
Routing:
- net VBUS: track 85.2 -> 82.9 mm
- net Net-(R2-Pad1): track 244.8 -> 246.3 mm
- net GND: track 21.3 -> 22.3 mm, vias 10 -> 135
