File: pancakexxl_pcb/PancakeXXL V2-rounded.kicad_pcb (KiCad board)
At the start: 2 copper layers, 246 x 83 mm, 119 parts, among them J1 Conn_01x04, SW1 Reset, SW2 Boot, U1 XC6206PxxxMR, U2 RP2040, U3 W25Q128JVS, Y1 ABM8-272-T3

Commit message: update after many month
Final design of the case,
Final plate design,
Final PCB for production,
And many more
Parts:
- renumbered SW2 to Boot, SW1 to Reset
Changed lines of the file:
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@@
 		(descr "ALPS 5.2mm Square Low-profile Type (Surface Mount) SKQG Series, With stem, http://www.alps.com/prod/info/E/HTML/Tact/SurfaceMount/SKQG/SKQGAFE010.html")
 		(tags "SPST Button Switch")
-		(property "Reference" "SW1"
+		(property "Reference" "Reset"
 			(at 0 3.6 0)
 			(layer "B.SilkS")
@@
 		(descr "ALPS 5.2mm Square Low-profile Type (Surface Mount) SKQG Series, With stem, http://www.alps.com/prod/info/E/HTML/Tact/SurfaceMount/SKQG/SKQGAFE010.html")
 		(tags "SPST Button Switch")
-		(property "Reference" "SW2"
+		(property "Reference" "Boot"
 			(at 0 3.6 0)
 			(layer "B.SilkS")
